Commit message: manipulador calculando a trajetória do braço porém com alguns bugs

File: software/src/Manipulador_moveit_config/config/Manipulador.ros2_control.xacro (robot description, xacro)
@@ -43,11 +43,4 @@
                 <state_interface name="velocity"/>
             </joint>
-            <joint name="garra_direita_to_garra_base">
-                <command_interface name="position"/>
-                <state_interface name="position">
-                  <param name="initial_value">${initial_positions['garra_direita_to_garra_base']}</param>
-                </state_interface>
-                <state_interface name="velocity"/>
-            </joint>
             <joint name="garra_esquerda_to_garra_base">
                 <command_interface name="position"/>
