Commit message: Update NAV: Cross-launch-pkgs working with any map in /simulation

File: software/src/base_description/urdf/Base.xacro (robot description, xacro)
@@ -4,4 +4,6 @@
 <xacro:include filename="$(find base_description)/urdf/Base.trans" />
 <xacro:include filename="$(find base_description)/urdf/Base.gazebo" />
+<link name="base_footprint">
+</link>
 <link name="base_link">
   <inertial>
@@ -104,4 +106,9 @@
   </collision>
 </link>
+<joint name="base_footprint_joint" type="fixed">
+    <origin rpy="0 0 0" xyz="0 0 0.010" />
+    <parent link="base_footprint" />
+    <child link="base_link" />
+</joint>
 <joint name="right_wheel_to_base" type="continuous">
   <origin xyz="0.12186 -0.211067 0.07" rpy="0 0 0"/>
