Commit message: Update: navigation pkg working in a test urdf

File: software/src/base_description/urdf/car.urdf (robot description, URDF)
Before this commit: robot box_bot, 20 links, 19 joints
Links:
- link base_link: geometry collision box size=0.256 0.150 0.065; visual mesh filename=src/base_description/meshes/cute_cube.dae scale=0.256 0.150 0.065
- link lidar_link: geometry collision box size=0.05 0.05 0.030; visual mesh filename=src/base_description/meshes/sensors/rplidar.dae scale=1.0 1.0 1.0
