Commit message: UPDATE: URDF with aligned wheels, but planar pluggin doesnt work pretty well

File: software/src/simulation_pkg/urdf/robot.xacro (robot description, xacro)
@@ -1,5 +1,5 @@
-<?xml version="1.0" ?>
+<?xml version="1.0"?>
 <robot name="robot" xmlns:xacro="http://www.ros.org/wiki/xacro">
-    <xacro:include filename="$(find simulation_pkg)/urdf/robot.gazebo"/>
+    <xacro:include filename="$(find simulation_pkg)/urdf/robot.gazebo" />
     <!-- root link, on the ground just below the model origin -->
     <link name="base_footprint">
@@ -12,5 +12,5 @@
     </link>
     <joint name="base_link_joint" type="fixed">
-        <origin xyz="0.0 0 1.25" rpy="0 0 0" />
+        <origin xyz="0.0 0 0.105" rpy="0 0 0" />
         <parent link="base_footprint" />
         <child link="base_link" />
@@ -18,10 +18,10 @@
     <link name="base_link">
         <visual>
-            <origin xyz="0.068650503425891296061 -0.083840399074440033478 0.040443740433454548888"
-                rpy="0 -0 0" />
-            <geometry>
-                <mesh filename="file://$(find simulation_pkg)/meshes/stl/lidar.stl" />
-            </geometry>
-            <material name="lidar_material">
+            <origin xyz="0.040970128253102346128 0.042066415995359325575 0.12400000000000016565"
+                rpy="3.141592653589793116 -0 2.7755575615628913511e-16" />
+            <geometry>
+                <mesh filename="file://$(find simulation_pkg)/meshes/stl/part_1.stl" />
+            </geometry>
+            <material name="part_1_material">
                 <color
                     rgba="0.61568627450980395466 0.81176470588235294379 0.92941176470588238168 1.0" />
@@ -29,71 +29,17 @@
         </visual>
         <collision>
-            <origin xyz="0.068650503425891296061 -0.083840399074440033478 0.040443740433454548888"
-                rpy="0 -0 0" />
-            <geometry>
-                <mesh filename="file://$(find simulation_pkg)/meshes/stl/lidar.stl" />
-            </geometry>
-        </collision>
-        <visual>
-            <origin xyz="0.11731235416125289361 0.15179281777659742181 -0.009556259566545493786"
-                rpy="0 -0 -0.52359877559829881566" />
-            <geometry>
-                <mesh filename="file://$(find simulation_pkg)/meshes/stl/perfil_colunas.stl" />
-            </geometry>
-            <material name="perfil_colunas_material">
-                <color
-                    rgba="0.90196078431372550543 0.90196078431372550543 0.90196078431372550543 1.0" />
-            </material>
-        </visual>
-        <collision>
-            <origin xyz="0.11731235416125289361 0.15179281777659742181 -0.009556259566545493786"
-                rpy="0 -0 -0.52359877559829881566" />
-            <geometry>
-                <mesh filename="file://$(find simulation_pkg)/meshes/stl/perfil_colunas.stl" />
-            </geometry>
-        </collision>
-        <visual>
-            <origin xyz="0.017124847813541788089 -0.021737033501267377655 0.034443740433454550498"
-                rpy="0 -0 0" />
-            <geometry>
-                <mesh filename="file://$(find simulation_pkg)/meshes/stl/mdf_motores.stl" />
-            </geometry>
-            <material name="mdf_motores_material">
-                <color
-                    rgba="0.90196078431372550543 0.83529411764705885357 0.6745098039215686736 1.0" />
-            </material>
-        </visual>
-        <collision>
-            <origin xyz="0.017124847813541788089 -0.021737033501267377655 0.034443740433454550498"
-                rpy="0 -0 0" />
-            <geometry>
-                <mesh filename="file://$(find simulation_pkg)/meshes/stl/mdf_motores.stl" />
-            </geometry>
-        </collision>
-        <visual>
-            <origin xyz="-0.18325016488188017316 -0.0217370335012673499 -0.009556259566545493786"
-                rpy="0 -0 1.57079632679489678" />
-            <geometry>
-                <mesh filename="file://$(find simulation_pkg)/meshes/stl/perfil_colunas.stl" />
-            </geometry>
-            <material name="perfil_colunas_material">
-                <color
-                    rgba="0.90196078431372550543 0.90196078431372550543 0.90196078431372550543 1.0" />
-            </material>
-        </visual>
-        <collision>
-            <origin xyz="-0.18325016488188017316 -0.0217370335012673499 -0.009556259566545493786"
-                rpy="0 -0 1.57079632679489678" />
-            <geometry>
-                <mesh filename="file://$(find simulation_pkg)/meshes/stl/perfil_colunas.stl" />
-            </geometry>
-        </collision>
-        <visual>
-            <origin xyz="0.070294802381689489024 -0.064708319082856041726 0.031443740433454547833"
-                rpy="0 -0 0" />
-            <geometry>
-                <mesh filename="file://$(find simulation_pkg)/meshes/stl/imu.stl" />
-            </geometry>
-            <material name="imu_material">
+            <origin xyz="0.040970128253102346128 0.042066415995359325575 0.12400000000000016565"
+                rpy="3.141592653589793116 -0 2.7755575615628913511e-16" />
+            <geometry>
+                <mesh filename="file://$(find simulation_pkg)/meshes/stl/part_1.stl" />
+            </geometry>
+        </collision>
+        <visual>
+            <origin xyz="0.038431848347187068382 -0.013246810296550448616 0.098000000000000142553"
+                rpy="0 -0 2.7755575615628913511e-16" />
+            <geometry>
+                <mesh filename="file://$(find simulation_pkg)/meshes/stl/part_2.stl" />
+            </geometry>
+            <material name="part_2_material">
                 <color
                     rgba="0.64705882352941179736 0.64705882352941179736 0.64705882352941179736 1.0" />
@@ -101,31 +47,31 @@
         </visual>
         <collision>
-            <origin xyz="0.070294802381689489024 -0.064708319082856041726 0.031443740433454547833"
-                rpy="0 -0 0" />
-            <geometry>
-                <mesh filename="file://$(find simulation_pkg)/meshes/stl/imu.stl" />
-            </geometry>
-        </collision>
-        <visual>
-            <origin xyz="0.11731235416125274096 -0.19526688477913226039 -0.009556259566545493786"
-                rpy="0 -0 -2.6179938779914944114" />
-            <geometry>
-                <mesh filename="file://$(find simulation_pkg)/meshes/stl/perfil_colunas.stl" />
-            </geometry>
-            <material name="perfil_colunas_material">
-                <color
-                    rgba="0.90196078431372550543 0.90196078431372550543 0.90196078431372550543 1.0" />
-            </material>
-        </visual>
-        <collision>
-            <origin xyz="0.11731235416125274096 -0.19526688477913226039 -0.009556259566545493786"
-                rpy="0 -0 -2.6179938779914944114" />
-            <geometry>
-                <mesh filename="file://$(find simulation_pkg)/meshes/stl/perfil_colunas.stl" />
-            </geometry>
-        </collision>
-        <visual>
-            <origin xyz="0.094662354161252709739 -0.15603593398769710632 -0.059198882331824187464"
-                rpy="0 -0 0.52359877559829881566" />
+            <origin xyz="0.038431848347187068382 -0.013246810296550448616 0.098000000000000142553"
+                rpy="0 -0 2.7755575615628913511e-16" />
+            <geometry>
+                <mesh filename="file://$(find simulation_pkg)/meshes/stl/part_2.stl" />
+            </geometry>
+        </collision>
+        <visual>
+            <origin xyz="-0.17959202910435595468 -0.10368750634771083108 -0.010000000000000000208"
+                rpy="0 -0 -1.0471975511965976313" />
+            <geometry>
+                <mesh filename="file://$(find simulation_pkg)/meshes/stl/perfil_motores.stl" />
+            </geometry>
+            <material name="perfil_motores_material">
+                <color
+                    rgba="0.90196078431372550543 0.90196078431372550543 0.90196078431372550543 1.0" />
+            </material>
+        </visual>
+        <collision>
+            <origin xyz="-0.17959202910435595468 -0.10368750634771083108 -0.010000000000000000208"
+                rpy="0 -0 -1.0471975511965976313" />
+            <geometry>
+                <mesh filename="file://$(find simulation_pkg)/meshes/stl/perfil_motores.stl" />
+            </geometry>
+        </collision>
+        <visual>
+            <origin xyz="0.13429890048642967315 -0.07753750634771117145 -0.043642622765278749064"
+                rpy="0 -0 1.0471975511965976313" />
             <geometry>
                 <mesh filename="file://$(find simulation_pkg)/meshes/stl/motor.stl" />
@@ -136,49 +82,30 @@
         </visual>
         <collision>
-            <origin xyz="0.094662354161252709739 -0.15603593398769710632 -0.059198882331824187464"
-                rpy="0 -0 0.52359877559829881566" />
-            <geometry>
-                <mesh filename="file://$(find simulation_pkg)/meshes/stl/motor.stl" />
-            </geometry>
-        </collision>
-        <visual>
-            <origin xyz="0.1208123541612529106 0.15785499560308846601 -0.025556259566545502793"
-                rpy="0 -0 2.6179938779914944114" />
-            <geometry>
-                <mesh filename="file://$(find simulation_pkg)/meshes/stl/perfil_motores.stl" />
-            </geometry>
-            <material name="perfil_motores_material">
-                <color
-                    rgba="0.90196078431372550543 0.90196078431372550543 0.90196078431372550543 1.0" />
-            </material>
-        </visual>
-        <collision>
-            <origin xyz="0.1208123541612529106 0.15785499560308846601 -0.025556259566545502793"
-                rpy="0 -0 2.6179938779914944114" />
-            <geometry>
-                <mesh filename="file://$(find simulation_pkg)/meshes/stl/perfil_motores.stl" />
-            </geometry>
-        </collision>
-        <visual>
-            <origin xyz="0.12081235416125274407 -0.20132906260562333234 -0.025556259566545502793"
-                rpy="0 -0 0.52359877559829881566" />
-            <geometry>
-                <mesh filename="file://$(find simulation_pkg)/meshes/stl/perfil_motores.stl" />
-            </geometry>
-            <material name="perfil_motores_material">
-                <color
-                    rgba="0.90196078431372550543 0.90196078431372550543 0.90196078431372550543 1.0" />
-            </material>
-        </visual>
-        <collision>
-            <origin xyz="0.12081235416125274407 -0.20132906260562333234 -0.025556259566545502793"
-                rpy="0 -0 0.52359877559829881566" />
-            <geometry>
-                <mesh filename="file://$(find simulation_pkg)/meshes/stl/perfil_motores.stl" />
-            </geometry>
-        </collision>
-        <visual>
-            <origin xyz="0.017124847813541788089 -0.021737033501267377655 -0.015556259566545493911"
-                rpy="0 -0 0" />
+            <origin xyz="0.13429890048642967315 -0.07753750634771117145 -0.043642622765278749064"
+                rpy="0 -0 1.0471975511965976313" />
+            <geometry>
+                <mesh filename="file://$(find simulation_pkg)/meshes/stl/motor.stl" />
+            </geometry>
+        </collision>
+        <visual>
+            <origin xyz="-0.17352985127786493824 -0.1001875063477108696 0.0060000000000000001249"
+                rpy="0 -0 -1.0471975511965976313" />
+            <geometry>
+                <mesh filename="file://$(find simulation_pkg)/meshes/stl/perfil_colunas.stl" />
+            </geometry>
+            <material name="perfil_colunas_material">
+                <color
+                    rgba="0.90196078431372550543 0.90196078431372550543 0.90196078431372550543 1.0" />
+            </material>
+        </visual>
+        <collision>
+            <origin xyz="-0.17352985127786493824 -0.1001875063477108696 0.0060000000000000001249"
+                rpy="0 -0 -1.0471975511965976313" />
+            <geometry>
+                <mesh filename="file://$(find simulation_pkg)/meshes/stl/perfil_colunas.stl" />
+            </geometry>
+        </collision>
+        <visual>
+            <origin xyz="0 0 0" rpy="0 -0 0" />
             <geometry>
                 <mesh filename="file://$(find simulation_pkg)/meshes/stl/mdf_motores.stl" />
@@ -190,6 +117,5 @@
         </visual>
         <collision>
-            <origin xyz="0.017124847813541788089 -0.021737033501267377655 -0.015556259566545493911"
-                rpy="0 -0 0" />
+            <origin xyz="0 0 0" rpy="0 -0 0" />
             <geometry>
                 <mesh filename="file://$(find simulation_pkg)/meshes/stl/mdf_motores.stl" />
@@ -197,24 +123,6 @@
         </collision>
         <visual>
-            <origin xyz="-0.19025016488188017938 -0.0217370335012673499 -0.025556259566545502793"
-                rpy="0 -0 -1.570796326794896558" />
-            <geometry>
-                <mesh filename="file://$(find simulation_pkg)/meshes/stl/perfil_motores.stl" />
-            </geometry>
-            <material name="perfil_motores_material">
-                <color
-                    rgba="0.90196078431372550543 0.90196078431372550543 0.90196078431372550543 1.0" />
-            </material>
-        </visual>
-        <collision>
-            <origin xyz="-0.19025016488188017938 -0.0217370335012673499 -0.025556259566545502793"
-                rpy="0 -0 -1.570796326794896558" />
-            <geometry>
-                <mesh filename="file://$(find simulation_pkg)/meshes/stl/perfil_motores.stl" />
-            </geometry>
-        </collision>
-        <visual>
-            <origin xyz="0.094662354161252904028 0.11256186698516235101 -0.059198882331824187464"
-                rpy="-5.5511151231257827021e-17 -0 2.6179938779914944114" />
+            <origin xyz="-0.13429890048642978417 -0.077537506347710782872 -0.043642622765278749064"
+                rpy="0 -0 -1.0471975511965976313" />
             <geometry>
                 <mesh filename="file://$(find simulation_pkg)/meshes/stl/motor.stl" />
@@ -225,13 +133,87 @@
         </visual>
         <collision>
-            <origin xyz="0.094662354161252904028 0.11256186698516235101 -0.059198882331824187464"
-                rpy="-5.5511151231257827021e-17 -0 2.6179938779914944114" />
-            <geometry>
-                <mesh filename="file://$(find simulation_pkg)/meshes/stl/motor.stl" />
-            </geometry>
-        </collision>
-        <visual>
-            <origin xyz="-0.13795016488188016623 -0.021737033501267322144 -0.059198882331824187464"
-                rpy="0 -0 -1.570796326794896558" />
+            <origin xyz="-0.13429890048642978417 -0.077537506347710782872 -0.043642622765278749064"
+                rpy="0 -0 -1.0471975511965976313" />
+            <geometry>
+                <mesh filename="file://$(find simulation_pkg)/meshes/stl/motor.stl" />
+            </geometry>
+        </collision>
+        <visual>
+            <origin xyz="0.17959202910435578815 -0.10368750634771116415 -0.010000000000000000208"
+                rpy="0 -0 1.0471975511965976313" />
+            <geometry>
+                <mesh filename="file://$(find simulation_pkg)/meshes/stl/perfil_motores.stl" />
+            </geometry>
+            <material name="perfil_motores_material">
+                <color
+                    rgba="0.90196078431372550543 0.90196078431372550543 0.90196078431372550543 1.0" />
+            </material>
+        </visual>
+        <collision>
+            <origin xyz="0.17959202910435578815 -0.10368750634771116415 -0.010000000000000000208"
+                rpy="0 -0 1.0471975511965976313" />
+            <geometry>
+                <mesh filename="file://$(find simulation_pkg)/meshes/stl/perfil_motores.stl" />
+            </geometry>
+        </collision>
+        <visual>
+            <origin xyz="2.498001805406602216e-16 0.20037501269542196125 0.0060000000000000001249"
+                rpy="0 -0 3.141592653589793116" />
+            <geometry>
+                <mesh filename="file://$(find simulation_pkg)/meshes/stl/perfil_colunas.stl" />
+            </geometry>
+            <material name="perfil_colunas_material">
+                <color
+                    rgba="0.90196078431372550543 0.90196078431372550543 0.90196078431372550543 1.0" />
+            </material>
+        </visual>
+        <collision>
+            <origin xyz="2.498001805406602216e-16 0.20037501269542196125 0.0060000000000000001249"
+                rpy="0 -0 3.141592653589793116" />
+            <geometry>
+                <mesh filename="file://$(find simulation_pkg)/meshes/stl/perfil_colunas.stl" />
+            </geometry>
+        </collision>
+        <visual>
+            <origin xyz="2.7755575615628913511e-16 0.20737501269542196747 -0.010000000000000000208"
+                rpy="0 -0 3.141592653589793116" />
+            <geometry>
+                <mesh filename="file://$(find simulation_pkg)/meshes/stl/perfil_motores.stl" />
+            </geometry>
+            <material name="perfil_motores_material">
+                <color
+                    rgba="0.90196078431372550543 0.90196078431372550543 0.90196078431372550543 1.0" />
+            </material>
+        </visual>
+        <collision>
+            <origin xyz="2.7755575615628913511e-16 0.20737501269542196747 -0.010000000000000000208"
+                rpy="0 -0 3.141592653589793116" />
+            <geometry>
+                <mesh filename="file://$(find simulation_pkg)/meshes/stl/perfil_motores.stl" />
+            </geometry>
+        </collision>
+        <visual>
+            <origin
+                xyz="2.7755575615628913511e-17 -6.9388939039072283776e-17 0.10300000000000014699"
+                rpy="0 -0 2.7755575615628913511e-16" />
+            <geometry>
+                <mesh filename="file://$(find simulation_pkg)/meshes/stl/mdf_motores.stl" />
+            </geometry>
+            <material name="mdf_motores_material">
+                <color
+                    rgba="0.90196078431372550543 0.83529411764705885357 0.6745098039215686736 1.0" />
+            </material>
+        </visual>
+        <collision>
+            <origin
+                xyz="2.7755575615628913511e-17 -6.9388939039072283776e-17 0.10300000000000014699"
+                rpy="0 -0 2.7755575615628913511e-16" />
+            <geometry>
+                <mesh filename="file://$(find simulation_pkg)/meshes/stl/mdf_motores.stl" />
+            </geometry>
+        </collision>
+        <visual>
+            <origin xyz="2.9143354396410359186e-16 0.15507501269542195432 -0.04364262276527871437"
+                rpy="0 -0 3.141592653589793116" />
             <geometry>
                 <mesh filename="file://$(find simulation_pkg)/meshes/stl/motor.stl" />
@@ -242,17 +224,35 @@
         </visual>
         <collision>
-            <origin xyz="-0.13795016488188016623 -0.021737033501267322144 -0.059198882331824187464"
-                rpy="0 -0 -1.570796326794896558" />
-            <geometry>
-                <mesh filename="file://$(find simulation_pkg)/meshes/stl/motor.stl" />
+            <origin xyz="2.9143354396410359186e-16 0.15507501269542195432 -0.04364262276527871437"
+                rpy="0 -0 3.141592653589793116" />
+            <geometry>
+                <mesh filename="file://$(find simulation_pkg)/meshes/stl/motor.stl" />
+            </geometry>
+        </collision>
+        <visual>
+            <origin xyz="0.17352985127786474395 -0.10018750634771117491 0.0060000000000000001249"
+                rpy="0 -0 1.0471975511965976313" />
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