Commit message: Update: Now robot.xacro receive parameters (use_time_sim) to separate when use real robot or simulated robot

File: software/src/omnicare_description/urdf/robot.xacro (robot description, xacro)
@@ -1,6 +1,13 @@
 <?xml version="1.0"?>
 <robot name="robot" xmlns:xacro="http://www.ros.org/wiki/xacro">
-    <xacro:include filename="$(find omnicare_description)/urdf/robot.gazebo" />
-    <!-- <xacro:include filename="$(find omnicare_description)/urdf/ros2_control.xacro"/> -->
+    <xacro:arg name="sim_mode" default="false" />
+    <xacro:if value="$(arg sim_mode)">
+        <xacro:include filename="$(find omnicare_description)/urdf/robot.gazebo" />
+    </xacro:if>
+    <xacro:unless value="$(arg sim_mode)">
+        <xacro:include filename="$(find omnicare_description)/urdf/ros2_control.xacro" />
+    </xacro:unless>
+    <!-- <xacro:include filename="$(find omnicare_description)/urdf/robot.gazebo" /> -->
+    <!-- <xacro:include filename="$(find omnicare_description)/urdf/ros2_control.xacro" /> -->
     <joint name="base_footprint_to_base_link" type="fixed">
         <parent link="base_footprint" />

File: software/src/omnicare_description/urdf/ros2_control.xacro (robot description, xacro)
@@ -1,85 +1,31 @@
 <?xml version="1.0"?>
 <robot xmlns:xacro="http://www.ros.org/wiki/xacro">
-    <!-- <ros2_control name="RealRobot" type="system">
+    <ros2_control name="RealRobot" type="system">
         <hardware>
             <plugin>omnidrive_stm32/OmniDriveSTM32</plugin>
-            <param name="left_wheel_name">left_wheel_joint</param>
-            <param name="right_wheel_name">right_wheel_joint</param>
-            <param name="back_wheel_name">back_wheel_joint</param>
+            <param name="left_wheel_name">wheel2_speed</param>
+            <param name="right_wheel_name">wheel1_speed</param>
+            <param name="back_wheel_name">wheel3_speed</param>
             <param name="loop_rate">30</param>
-            <param name="device">/dev/ttyUSB0</param>
+            <param name="device">/dev/ttyACM0</param>
             <param name="baud_rate">115200</param>
-            <param name="timeout">1000</param>
-            <param name="enc_counts_per_rev">3436</param>
-        </hardware>
-        <joint name="right_wheel_to_base">
-            <command_interface name="velocity">
-                <param name="min">-10</param>
-                <param name="max">10</param>
-            </command_interface>
-            <state_interface name="velocity"/>
-            <state_interface name="position"/>
-        </joint>
-        <joint name="left_wheel_to_base">
-            <command_interface name="velocity">
-                <param name="min">-10</param>
-                <param name="max">10</param>
-            </command_interface>
-            <state_interface name="velocity"/>
-            <state_interface name="position"/>
-        </joint>
-        <joint name="back_wheel_to_base">
-            <command_interface name="velocity">
-                <param name="min">-10</param>
-                <param name="max">10</param>
-            </command_interface>
-            <state_interface name="velocity"/>
-            <state_interface name="position"/>
-        </joint>
-    </ros2_control> -->
-    <ros2_control name="GazeboSystem" type="system">
-        <hardware>
-            <plugin>gazebo_ros2_control/GazeboSystem</plugin>
+            <param name="timeout_ms">1000</param>
+            <param name="enc_counts_per_rev">12770</param>
         </hardware>
         <joint name="wheel1_speed">
-            <command_interface name="velocity">
-                <param name="min">-10</param>
-                <param name="max">10</param>
-            </command_interface>
+            <command_interface name="velocity" />
+            <state_interface name="position" />
             <state_interface name="velocity" />
-            <state_interface name="position" />
         </joint>
         <joint name="wheel2_speed">
-            <command_interface name="velocity">
-                <param name="min">-10</param>
-                <param name="max">10</param>
-            </command_interface>
+            <command_interface name="velocity" />
+            <state_interface name="position" />
             <state_interface name="velocity" />
-            <state_interface name="position" />
         </joint>
         <joint name="wheel3_speed">
-            <command_interface name="velocity">
-                <param name="min">-10</param>
-                <param name="max">10</param>
-            </command_interface>
+            <command_interface name="velocity" />
+            <state_interface name="position" />
             <state_interface name="velocity" />
-            <state_interface name="position" />
         </joint>
     </ros2_control>
-    <gazebo>
-        <plugin filename="libgazebo_ros2_control.so" name="gazebo_ros2_control">
-            <robot_param>robot_description</robot_param>
-            <robot_param_node>robot_state_publisher</robot_param_node>
-            <parameters>$(find omnicare_control_pkg)/config/ros2_control/omnidirectional_controller.yaml</parameters>
-        </plugin>
-        <!-- <plugin filename="libgazebo_ros_p3d.so" name="gazebo_ros_p3d">
-            <ros>
-                <namespace>gazebo_ground_truth</namespace>
-            </ros>
-            <frame_name>world</frame_name>
-            <body_name>base_link</body_name>
-            <update_rate>50.0</update_rate>
-            <gaussian_noise>0.01</gaussian_noise>
-        </plugin> -->
-    </gazebo>
 </robot>

Commit message: Update&Add: Update the XACRO of the robot (LiDAR link for real LiDAR) && Add Teleop Joy launch

File: software/src/omnicare_description/urdf/robot.xacro (robot description, xacro)
@@ -8,6 +8,10 @@
         <xacro:include filename="$(find omnicare_description)/urdf/ros2_control.xacro" />
     </xacro:unless>
-    <!-- <xacro:include filename="$(find omnicare_description)/urdf/robot.gazebo" /> -->
-    <!-- <xacro:include filename="$(find omnicare_description)/urdf/ros2_control.xacro" /> -->
+    <link name="lidar_link"></link>
+    <joint name="lidar_to_base" type="fixed">
+        <parent link="base_link" />
+        <child link="lidar_link" />
+        <origin rpy="0.0 0 3.14" xyz="0 0 0" />
+    </joint>
     <joint name="base_footprint_to_base_link" type="fixed">
         <parent link="base_footprint" />
